Commit message: ur5.urdf

File: meshes/ur5/visual/ur5.urdf (robot description, URDF)
Before this commit: robot ur5, 11 links, 10 joints
Links:
- removed link forearm01_link
- added link forearm02_link; collision mesh filename=forearm02.obj; visual mesh filename=forearm02.obj
- added link forearm03_01_link; collision mesh filename=forearm03_01.obj; visual mesh filename=forearm03_01.obj
- added link forearm03_link; collision mesh filename=forearm03.obj; visual mesh filename=forearm03.obj
- added link forearm_link, mass 2.275; collision mesh filename=forearm.obj; visual mesh filename=forearm.obj
- added link shoulder02_link; collision mesh filename=shoulder02.obj; visual mesh filename=shoulder02.obj
- added link upper_arm02_link; collision mesh filename=upperarm02.obj; visual mesh filename=upperarm02.obj
- added link upper_arm03_01_link; collision mesh filename=upperarm03_01.obj; visual mesh filename=upperarm03_01.obj
- added link upper_arm03_link; collision mesh filename=upperarm03.obj; visual mesh filename=upperarm03.obj
- added link upper_arm_01_link; collision mesh filename=upperarm_01.obj; visual mesh filename=upperarm_01.obj
- added link wrist_1_01_link; collision mesh filename=wrist1_01.obj; visual mesh filename=wrist1_01.obj
- added link wrist_2_01_link; collision mesh filename=wrist2_01.obj; visual mesh filename=wrist2_01.obj
- link base_link: geometry collision mesh filename=base.obj; visual mesh filename=base.obj
- link shoulder_link: geometry collision mesh filename=shoulder.obj; visual mesh filename=shoulder.obj
- link upper_arm_link: geometry collision mesh filename=upperarm.obj; visual mesh filename=upperarm.obj
- link wrist_1_link: geometry collision mesh filename=wrist1.obj; visual mesh filename=wrist1.obj
- link wrist_2_link: geometry collision mesh filename=wrist2.obj; visual mesh filename=wrist2.obj
- link wrist_3_link: geometry collision mesh filename=wrist3.obj; visual mesh filename=wrist3.obj
Joints:
- added joint elbow_fix02_joint: type fixed, parent forearm_link, child forearm02_link
- added joint elbow_fix03_01_joint: type fixed, parent forearm_link, child forearm03_01_link
- added joint elbow_fix03_joint: type fixed, parent forearm_link, child forearm03_link
- added joint shoulder_lift_fix02_joint: type fixed, parent upper_arm_link, child upper_arm02_link
- added joint shoulder_lift_fix03_01_joint: type fixed, parent upper_arm_link, child upper_arm03_01_link
- added joint shoulder_lift_fix03_joint: type fixed, parent upper_arm_link, child upper_arm03_link
- added joint shoulder_lift_fix_01_joint: type fixed, parent upper_arm_link, child upper_arm_01_link
- added joint shoulder_pan_fix_joint: type fixed, parent shoulder_link, child shoulder02_link
- added joint wrist_1_fix_joint: type fixed, parent wrist_1_link, child wrist_1_01_link
- added joint wrist_2_fix_joint: type fixed, parent wrist_2_link, child wrist_2_01_link
- joint elbow_joint: child forearm01_link -> forearm_link
- joint wrist_1_joint: parent forearm01_link -> forearm_link

File: urdf/ur5(复件).urdf (robot description, URDF)
Before this commit: robot ur5, 11 links, 10 joints
Links:
- removed link forearm01_link
- added link forearm_link, mass 2.275; collision mesh filename=/home/tungkw/download/universal_robot-melodic-devel/ur_desc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; visual mesh filename=/home/tungkw/download/universal_robot-melodic-devel/ur_desc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
Joints:
- joint elbow_joint: child forearm01_link -> forearm_link
- joint wrist_1_joint: parent forearm01_link -> forearm_link
