Commit message: 'finished'

File: meshes/ur5/ur5.urdf (robot description, URDF)
Before this commit: robot ur5, 11 links, 10 joints
Links:
- removed link forearm01_link
- added link forearm02_link, mass 0.0; collision mesh filename=forearm02.obj; visual mesh filename=forearm02.obj
- added link forearm03_01_link, mass 0.0; collision mesh filename=forearm03_01.obj; visual mesh filename=forearm03_01.obj
- added link forearm03_link, mass 0.0; collision mesh filename=forearm03.obj; visual mesh filename=forearm03.obj
- added link forearm_link, mass 2.275; collision mesh filename=forearm.obj; visual mesh filename=forearm.obj
- added link shoulder02_link, mass 0.0; collision mesh filename=shoulder02.obj; visual mesh filename=shoulder02.obj
- added link upper_arm02_link, mass 0.0; collision mesh filename=upperarm02.obj; visual mesh filename=upperarm02.obj
- added link upper_arm03_01_link, mass 0.0; collision mesh filename=upperarm03_01.obj; visual mesh filename=upperarm03_01.obj
- added link upper_arm03_link, mass 0.0; collision mesh filename=upperarm03.obj; visual mesh filename=upperarm03.obj
- added link upper_arm_01_link, mass 0.0; collision mesh filename=upperarm_01.obj; visual mesh filename=upperarm_01.obj
- added link wrist_1_01_link, mass 0.0; collision mesh filename=wrist1_01.obj; visual mesh filename=wrist1_01.obj
- added link wrist_2_01_link, mass 0.0; collision mesh filename=wrist2_01.obj; visual mesh filename=wrist2_01.obj
- link base: mass None -> 0.0
- link base_link: geometry collision mesh filename=base.obj; visual mesh filename=base.obj
- link ee_link: mass None -> 0.0
- link shoulder_link: geometry collision mesh filename=shoulder.obj; visual mesh filename=shoulder.obj
- link tool0: mass None -> 0.0
- link upper_arm_link: geometry collision mesh filename=upperarm.obj; visual mesh filename=upperarm.obj
- link wrist_1_link: geometry collision mesh filename=wrist1.obj; visual mesh filename=wrist1.obj
- link wrist_2_link: geometry collision mesh filename=wrist2.obj; visual mesh filename=wrist2.obj
- link wrist_3_link: geometry collision mesh filename=wrist3.obj; visual mesh filename=wrist3.obj
Joints:
- added joint elbow_fix02_joint: type fixed, parent forearm_link, child forearm02_link
- added joint elbow_fix03_01_joint: type fixed, parent forearm_link, child forearm03_01_link
- added joint elbow_fix03_joint: type fixed, parent forearm_link, child forearm03_link
- added joint shoulder_lift_fix02_joint: type fixed, parent upper_arm_link, child upper_arm02_link
- added joint shoulder_lift_fix03_01_joint: type fixed, parent upper_arm_link, child upper_arm03_01_link
- added joint shoulder_lift_fix03_joint: type fixed, parent upper_arm_link, child upper_arm03_link
- added joint shoulder_lift_fix_01_joint: type fixed, parent upper_arm_link, child upper_arm_01_link
- added joint shoulder_pan_fix_joint: type fixed, parent shoulder_link, child shoulder02_link
- added joint wrist_1_fix_joint: type fixed, parent wrist_1_link, child wrist_1_01_link
- added joint wrist_2_fix_joint: type fixed, parent wrist_2_link, child wrist_2_01_link
- joint elbow_joint: child forearm01_link -> forearm_link
- joint wrist_1_joint: parent forearm01_link -> forearm_link

Commit message: inverse

File: meshes/ur5/ur5.urdf (robot description, URDF)
Before this commit: robot ur5, 21 links, 20 joints
Links:
- link base_link: geometry collision mesh filename=collision/base.stl; visual mesh filename=base.obj
- link shoulder02_link: geometry visual mesh filename=shoulder02.obj
- link shoulder_link: geometry collision mesh filename=collision/shoulder.stl; visual mesh filename=shoulder.obj
